File: signalbuffer_single/signalbuffer_single.sch (KiCad schematic (older format))
At the start: 13 parts, among them J1 GND in, J2 VDD in, J3 VSS in, J4 Signal gnd, J6 Signal In, J7 Bias In, J9 Signal out, U1 LM318N

Commit message: updates
Parts:
- added C1: C_Small, symbol C_Small
- U1: symbol LM318N -> LM318N-RESCUE-signalbuffer_single
Connections:
- net at J9.1 (Pin_1), R9.1, U1.6: now also C1.1
- net at R7.1, R9.2, U1.2 (-): now also C1.2
Changed lines of the file:
@@
 EESchema Schematic File Version 2
+LIBS:signalbuffer_single-rescue
 LIBS:power
 LIBS:device
 LIBS:switches
 LIBS:relays
-LIBS:motors
 LIBS:transistors
 LIBS:conn
@@
 LIBS:contrib
 LIBS:valves
+LIBS:signalbuffer_single-cache
 EELAYER 25 0
 EELAYER END
@@
 	5650 3900 6050 3900
 Wire Wire Line
-	6050 3900 6050 3450
+	6050 3450 6050 4150
 Connection ~ 6050 3450
 Wire Wire Line
@@
 $EndComp
 $Comp
-L LM318N U1
+L LM318N-RESCUE-signalbuffer_single U1
 U 1 1 5AA8F957
 P 5650 3450
@@
 	4800 3900 5000 3900
 Wire Wire Line
+	5350 3550 5350 4150
+$Comp
+L C_Small C1
+U 1 1 5B2FE5DA
+P 5500 4150
+F 0 "C1" H 5510 4220 50  0000 L CNN
+F 1 "C_Small" H 5510 4070 50  0000 L CNN
+F 2 "" H 5500 4150 50  0000 C CNN
+F 3 "" H 5500 4150 50  0000 C CNN
+	1    5500 4150
+	0    1    1    0
+$EndComp
+Wire Wire Line
+	5350 4150 5400 4150
+Connection ~ 5350 3900
+Wire Wire Line
+	6050 4150 5600 4150
+Connection ~ 6050 3900
+Wire Wire Line
 	6750 3850 6750 3750
 Wire Wire Line
 	6750 3750 6900 3750
-Wire Wire Line
-	5350 3550 5350 3900
 $EndSCHEMATC
