File: signal_mover/signal_mover.sch (KiCad schematic (older format))
At the start: 4 parts

Commit message: updated signal mover
Parts:
- P1: renamed from P?; footprint (none) -> Connector_PinSocket_2.54mm:PinSocket_1x03_P2.54mm_Vertical; symbol CONN_01X03 -> signal_mover-rescue:CONN_01X03
- R1, R2: renamed from R?; footprint (none) -> Resistor_THT:R_Axial_DIN0207_L6.3mm_D2.5mm_P7.62mm_Horizontal; symbol R -> signal_mover-rescue:R
- RV1: renamed from RV?; footprint (none) -> Potentiometer_THT:Potentiometer_Piher_PC-16_Single_Vertical; symbol POT -> signal_mover-rescue:POT
Changed lines of the file:
@@
-EESchema Schematic File Version 2
-LIBS:power
-LIBS:device
-LIBS:transistors
-LIBS:conn
-LIBS:linear
-LIBS:regul
-LIBS:74xx
-LIBS:cmos4000
-LIBS:adc-dac
-LIBS:memory
-LIBS:xilinx
-LIBS:microcontrollers
-LIBS:dsp
-LIBS:microchip
-LIBS:analog_switches
-LIBS:motorola
-LIBS:texas
-LIBS:intel
-LIBS:audio
-LIBS:interface
-LIBS:digital-audio
-LIBS:philips
-LIBS:display
-LIBS:cypress
-LIBS:siliconi
-LIBS:opto
-LIBS:atmel
-LIBS:contrib
-LIBS:valves
-EELAYER 25 0
+EESchema Schematic File Version 4
+LIBS:signal_mover-cache
+EELAYER 26 0
 EELAYER END
 $Descr A4 11693 8268
@@
 $EndDescr
 $Comp
-L POT RV?
+L signal_mover-rescue:POT RV1
 U 1 1 5BC4D0BE
 P 3850 3250
-F 0 "RV?" H 3850 3170 50  0000 C CNN
+F 0 "RV1" H 3850 3170 50  0000 C CNN
 F 1 "POT" H 3850 3250 50  0000 C CNN
-F 2 "" H 3850 3250 50  0000 C CNN
+F 2 "Potentiometer_THT:Potentiometer_Piher_PC-16_Single_Vertical" H 3850 3250 50  0001 C CNN
 F 3 "" H 3850 3250 50  0000 C CNN
 	1    3850 3250
@@
 $EndComp
 $Comp
-L R R?
+L signal_mover-rescue:R R1
 U 1 1 5BC4D184
 P 4150 3000
-F 0 "R?" V 4230 3000 50  0000 C CNN
+F 0 "R1" V 4230 3000 50  0000 C CNN
 F 1 "R" V 4150 3000 50  0000 C CNN
-F 2 "" V 4080 3000 50  0000 C CNN
+F 2 "Resistor_THT:R_Axial_DIN0207_L6.3mm_D2.5mm_P7.62mm_Horizontal" V 4080 3000 50  0001 C CNN
 F 3 "" H 4150 3000 50  0000 C CNN
 	1    4150 3000
@@
 $EndComp
 $Comp
-L R R?
+L signal_mover-rescue:R R2
 U 1 1 5BC4D1C5
 P 4150 3500
-F 0 "R?" V 4230 3500 50  0000 C CNN
+F 0 "R2" V 4230 3500 50  0000 C CNN
 F 1 "R" V 4150 3500 50  0000 C CNN
-F 2 "" V 4080 3500 50  0000 C CNN
+F 2 "Resistor_THT:R_Axial_DIN0207_L6.3mm_D2.5mm_P7.62mm_Horizontal" V 4080 3500 50  0001 C CNN
 F 3 "" H 4150 3500 50  0000 C CNN
 	1    4150 3500
@@
 $EndComp
 $Comp
-L CONN_01X03 P?
+L signal_mover-rescue:CONN_01X03 P1
 U 1 1 5BC4D1F4
 P 4700 3250
-F 0 "P?" H 4700 3450 50  0000 C CNN
+F 0 "P1" H 4700 3450 50  0000 C CNN
 F 1 "CONN_01X03" V 4800 3250 50  0000 C CNN
-F 2 "" H 4700 3250 50  0000 C CNN
+F 2 "Connector_PinSocket_2.54mm:PinSocket_1x03_P2.54mm_Vertical" H 4700 3250 50  0001 C CNN
 F 3 "" H 4700 3250 50  0000 C CNN
 	1    4700 3250
