File: micpreamp/micpreamp.sch (KiCad schematic (older format))
At the start: 17 parts, among them J1 Input, J2 Output, J3 Vdd, J4 Gnd, U1 3.3 reg, U2 LM358

Commit message: added tiny spi proj and fixed an error with the mic preamp
Connections:
- net GND: no longer R1.1
- net at C1.1, R2.1, U1.2 (VO)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: now also R1.1
Changed lines of the file:
@@
 	3150 2300 3400 2300
 Wire Wire Line
-	3400 2300 3850 2300
+	3400 2300 3650 2300
 Connection ~ 3400 2300
 Wire Wire Line
@@
 Wire Wire Line
 	2250 2300 2550 2300
-Wire Wire Line
-	3400 3200 3400 2600
-Connection ~ 3400 2600
 Wire Wire Line
 	3400 3850 3400 3500
@@
 	5750 3750 6350 3750
 Connection ~ 5750 3750
+Wire Wire Line
+	3400 3200 3650 3200
+Wire Wire Line
+	3650 3200 3650 2300
+Connection ~ 3650 2300
+Wire Wire Line
+	3650 2300 3850 2300
 $EndSCHEMATC
