File: distpedal/distpedal.kicad_pcb (KiCad board)
At the start: 2 copper layers, 65.3 x 48.5 mm, 27 parts, among them J1 Insleeve, J2 Intip, J3 9vin, J4 gnd in, J5 Led+, J6 Led-, J7 Outtip, J8 Outsleve, U1 lm741

Commit message: some updates
Parts:
- moved R1 7.62 mm to (126.0, 81.3), turned to 180 degrees
- moved C2 5.06 mm to (119.6, 76.5), turned to 0 degrees
- moved R4 3.39 mm to (156.0, 85.9)
- moved J5 2.54 mm to (163.1, 90.7)
- moved C3 1.85 mm to (150.9, 72.4)
- moved R5 1.78 mm to (152.7, 103.6)
- moved C5 1.63 mm to (141.0, 100.6)
- moved D2 1.27 mm to (135.9, 95.5)
- moved D1 1.02 mm to (143.5, 90.9)
Routing:
- net Net-(C5-Pad1): track 46.5 -> 54.2 mm
- net Net-(R1-Pad1): track 29.4 -> 21.7 mm
- net Net-(C4-Pad2): track 22.5 -> 25.5 mm
- net Net-(C3-Pad1): track 18.7 -> 21.4 mm
- net Net-(C1-Pad2): track 22.6 -> 20.4 mm
- net Net-(C3-Pad2): track 5.41 -> 7.40 mm
- net Net-(J5-Pad1): track 7.99 -> 6.94 mm
- net GNDREF: track 187.0 -> 186.2 mm
- net Net-(C4-Pad1): track 5.33 -> 6.07 mm
