File: tiny85 spi controller/tiny85 spi controller.sch (KiCad schematic (older format))
At the start: 11 parts, among them J1 rs232, J3 ISP, SW1 SW_Push, U1 MAX232, U2 ATtiny85V-10SU

Commit message: some updates
Parts:
- J3: footprint Connector_PinSocket_2.54mm:PinSocket_2x03_P2.54mm_Vertical -> Connector_PinHeader_2.54mm:PinHeader_2x03_P2.54mm_Vertical
Changed lines of the file:
@@
 EESchema Schematic File Version 4
+LIBS:tiny85 spi controller-cache
 EELAYER 26 0
 EELAYER END
@@
 F 0 "J3" H 7400 2217 50  0000 C CNN
 F 1 "ISP" H 7400 2126 50  0000 C CNN
-F 2 "Connector_PinSocket_2.54mm:PinSocket_2x03_P2.54mm_Vertical" H 7350 1900 50  0001 C CNN
+F 2 "Connector_PinHeader_2.54mm:PinHeader_2x03_P2.54mm_Vertical" H 7350 1900 50  0001 C CNN
 F 3 "~" H 7350 1900 50  0001 C CNN
 	1    7350 1900
