File: numitron clock/numitron clock-rotated-numitrons.kicad_pcb (KiCad board)
At the start: 2 copper layers, 120 x 50.2 mm, 24 parts, among them J1 AVR-ISP-6, J2 rtc, J3 5v in, J4 UART, SW1 RST, SW2 Set M, SW3 Set H, U1 TPIC6595, U2 TPIC6595, U3 TPIC6595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

Commit message: work on numitron
Parts:
- turned NU1 to 180 degrees
- turned NU2 to 180 degrees
- turned NU3 to 180 degrees
- turned NU4 to 180 degrees
Routing:
- net VCC: track 288.5 -> 324.8 mm
- net Net-(U2-Pad4): track 21.2 -> 37.7 mm
- net Net-(U2-Pad14): track 37.9 -> 24.4 mm
- net Net-(U4-Pad7): track 34.0 -> 21.3 mm
- net Net-(U4-Pad4): track 20.6 -> 33.2 mm
- net Net-(U2-Pad17): track 12.1 -> 23.1 mm
- net Net-(NU1-Pad2): track 31.9 -> 21.2 mm
- net Net-(NU1-Pad4): track 24.1 -> 34.7 mm
- net Net-(NU1-Pad5): track 20.7 -> 30.2 mm, vias 0 -> 1
- net Net-(U4-Pad6): track 34.0 -> 24.6 mm, vias 0 -> 2
- net Net-(NU3-Pad2): track 30.7 -> 21.4 mm
- net Net-(U2-Pad7): track 33.1 -> 23.8 mm
- net Net-(NU1-Pad3): track 34.3 -> 26.4 mm, vias 0 -> 2
- net Net-(U2-Pad5): track 27.6 -> 35.3 mm
- net Net-(U4-Pad17): track 20.9 -> 13.7 mm
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