File: numitron clock/numitron clock.kicad_sch (KiCad schematic)
At the start: 24 parts, among them J1 AVR-ISP-6, J2 rtc, J3 5v in, J4 UART, SW1 RST, SW2 Set M, SW3 Set H, U1 TPIC6595, U10 Numitron_IV-9, U12 Numitron_IV-9, U2 TPIC6595, U22 Numitron_IV-9, U3 TPIC6595, U4 TPIC6595, U5 ATmega8L-8A, U9 Numitron_IV-9, Y1 Crystal

Commit message: work on numitron
Parts:
- renumbered U12 to NU1, U22 to NU2, U10 to NU3, U9 to NU4, U3 to U1, U1 to U2, U2 to U3
Changed lines of the file:
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@@
   (symbol (lib_id "numitron:Numitron_IV-9-Display") (at 179.07 59.69 270) (unit 1)
     (in_bom yes) (on_board yes)
-    (property "Reference" "U22" (id 0) (at 186.0042 59.69 0))
-    (property "Value" "Numitron_IV-9" (id 1) (at 188.3156 59.69 0))
+    (property "Reference" "NU2" (id 0) (at 172.72 59.69 0))
+    (property "Value" "Numitron_IV-9" (id 1) (at 170.18 58.42 0))
     (property "Footprint" "Numitron:numitron iv-9" (id 2) (at 163.83 59.69 0)
       (effects (font (size 1.27 1.27)) hide)
@@
   (symbol (lib_id "Interface_Expansion:TPIC6595") (at 148.59 58.42 0) (unit 1)
     (in_bom yes) (on_board yes)
-    (property "Reference" "U1" (id 0) (at 148.59 38.5826 0))
+    (property "Reference" "U2" (id 0) (at 148.59 38.5826 0))
     (property "Value" "TPIC6595" (id 1) (at 148.59 40.894 0))
     (property "Footprint" "Package_DIP:DIP-20_W7.62mm_LongPads" (id 2) (at 165.1 74.93 0)
@@
   (symbol (lib_id "numitron:Numitron_IV-9-Display") (at 242.57 101.6 270) (unit 1)
     (in_bom yes) (on_board yes)
-    (property "Reference" "U9" (id 0) (at 235.6358 101.6 0))
+    (property "Reference" "NU4" (id 0) (at 235.6358 101.6 0))
     (property "Value" "Numitron_IV-9" (id 1) (at 233.3244 101.6 0))
     (property "Footprint" "Numitron:numitron iv-9" (id 2) (at 227.33 101.6 0)
@@
   (symbol (lib_id "numitron:Numitron_IV-9-Display") (at 245.11 57.15 270) (unit 1)
     (in_bom yes) (on_board yes)
-    (property "Reference" "U10" (id 0) (at 238.1758 57.15 0))
-    (property "Value" "Numitron_IV-9" (id 1) (at 235.8644 57.15 0))
+    (property "Reference" "NU3" (id 0) (at 238.1758 57.15 0))
+    (property "Value" "Numitron_IV-9" (id 1) (at 236.22 55.88 0))
     (property "Footprint" "Numitron:numitron iv-9" (id 2) (at 229.87 57.15 0)
       (effects (font (size 1.27 1.27)) hide)
@@
   (symbol (lib_id "numitron:Numitron_IV-9-Display") (at 179.07 100.33 270) (unit 1)
     (in_bom yes) (on_board yes)
-    (property "Reference" "U12" (id 0) (at 172.1358 100.33 0))
+    (property "Reference" "NU1" (id 0) (at 172.1358 100.33 0))
     (property "Value" "Numitron_IV-9" (id 1) (at 169.8244 100.33 0))
     (property "Footprint" "Numitron:numitron iv-9" (id 2) (at 163.83 100.33 0)
@@
   (symbol (lib_id "Interface_Expansion:TPIC6595") (at 212.09 58.42 0) (unit 1)
     (in_bom yes) (on_board yes)
-    (property "Reference" "U2" (id 0) (at 212.09 38.5826 0))
+    (property "Reference" "U3" (id 0) (at 212.09 38.5826 0))
     (property "Value" "TPIC6595" (id 1) (at 212.09 40.894 0))
     (property "Footprint" "Package_DIP:DIP-20_W7.62mm_LongPads" (id 2) (at 228.6 74.93 0)
@@
   (symbol (lib_id "Interface_Expansion:TPIC6595") (at 148.59 100.33 0) (unit 1)
     (in_bom yes) (on_board yes)
-    (property "Reference" "U3" (id 0) (at 148.59 80.4926 0))
+    (property "Reference" "U1" (id 0) (at 148.59 80.4926 0))
     (property "Value" "TPIC6595" (id 1) (at 148.59 82.804 0))
     (property "Footprint" "Package_DIP:DIP-20_W7.62mm_LongPads" (id 2) (at 165.1 116.84 0)
@@
   )
   (symbol (lib_id "power:GNDREF") (at 146.05 77.47 0) (unit 1)
-    (in_bom yes) (on_board yes) (fields_autoplaced)
+    (in_bom yes) (on_board yes)
     (property "Reference" "#PWR04" (id 0) (at 146.05 83.82 0)
       (effects (font (size 1.27 1.27)) hide)
     )
-    (property "Value" "GNDREF" (id 1) (at 146.05 82.0325 0))
+    (property "Value" "GNDREF" (id 1) (at 140.97 80.01 0))
     (property "Footprint" "" (id 2) (at 146.05 77.47 0)
       (effects (font (size 1.27 1.27)) hide)
@@
   )
   (symbol (lib_id "power:GNDREF") (at 209.55 77.47 0) (unit 1)
-    (in_bom yes) (on_board yes) (fields_autoplaced)
+    (in_bom yes) (on_board yes)
     (property "Reference" "#PWR06" (id 0) (at 209.55 83.82 0)
       (effects (font (size 1.27 1.27)) hide)
     )
-    (property "Value" "GNDREF" (id 1) (at 209.55 82.0325 0))
+    (property "Value" "GNDREF" (id 1) (at 203.2 78.74 0))
     (property "Footprint" "" (id 2) (at 209.55 77.47 0)
       (effects (font (size 1.27 1.27)) hide)
@@
   )
   (symbol (lib_id "power:PWR_FLAG") (at 132.08 36.83 180) (unit 1)
-    (in_bom yes) (on_board yes) (fields_autoplaced)
+    (in_bom yes) (on_board yes)
     (property "Reference" "#FLG0102" (id 0) (at 132.08 38.735 0)
       (effects (font (size 1.27 1.27)) hide)
     )
-    (property "Value" "PWR_FLAG" (id 1) (at 132.08 41.3925 0))
+    (property "Value" "PWR_FLAG" (id 1) (at 138.43 38.1 0))
     (property "Footprint" "" (id 2) (at 132.08 36.83 0)
       (effects (font (size 1.27 1.27)) hide)
@@
   )
   (symbol (lib_id "Device:LED") (at 152.4 17.78 180) (unit 1)
-    (in_bom yes) (on_board yes) (fields_autoplaced)
-    (property "Reference" "D1" (id 0) (at 153.9875 11.6545 0))
-    (property "Value" "LED" (id 1) (at 153.9875 14.4296 0))
+    (in_bom yes) (on_board yes)
+    (property "Reference" "D1" (id 0) (at 154.94 15.24 0))
+    (property "Value" "LED" (id 1) (at 151.13 15.24 0))
     (property "Footprint" "LED_THT:LED_D5.0mm" (id 2) (at 152.4 17.78 0)
       (effects (font (size 1.27 1.27)) hide)
@@
   )
   (symbol (lib_id "Device:R") (at 143.51 17.78 90) (unit 1)
-    (in_bom yes) (on_board yes) (fields_autoplaced)
-    (property "Reference" "R2" (id 0) (at 143.51 12.7975 90))
+    (in_bom yes) (on_board yes)
+    (property "Reference" "R2" (id 0) (at 143.51 17.78 90))
     (property "Value" "R" (id 1) (at 143.51 15.5726 90))
     (property "Footprint" "Resistor_THT:R_Axial_DIN0207_L6.3mm_D2.5mm_P7.62mm_Horizontal" (id 2) (at 143.51 19.558 90)
@@
   )
   (symbol (lib_id "Device:LED") (at 152.4 21.59 180) (unit 1)
-    (in_bom yes) (on_board yes) (fields_autoplaced)
-    (property "Reference" "D2" (id 0) (at 153.9875 15.4645 0))
-    (property "Value" "LED" (id 1) (at 153.9875 18.2396 0))
+    (in_bom yes) (on_board yes)
+    (property "Reference" "D2" (id 0) (at 153.67 24.13 0))
+    (property "Value" "LED" (id 1) (at 153.67 26.67 0))
     (property "Footprint" "LED_THT:LED_D5.0mm" (id 2) (at 152.4 21.59 0)
       (effects (font (size 1.27 1.27)) hide)
@@
   )
   (symbol (lib_id "power:GNDREF") (at 129.54 36.83 0) (unit 1)
-    (in_bom yes) (on_board yes) (fields_autoplaced)
+    (in_bom yes) (on_board yes)
     (property "Reference" "#PWR0103" (id 0) (at 129.54 43.18 0)
       (effects (font (size 1.27 1.27)) hide)
     )
-    (property "Value" "GNDREF" (id 1) (at 129.54 41.3925 0))
+    (property "Value" "GNDREF" (id 1) (at 124.46 39.37 0))
     (property "Footprint" "" (id 2) (at 129.54 36.83 0)
       (effects (font (size 1.27 1.27)) hide)
@@
   )
   (symbol (lib_id "power:PWR_FLAG") (at 130.81 31.75 0) (unit 1)
-    (in_bom yes) (on_board yes) (fields_autoplaced)
+    (in_bom yes) (on_board yes)
     (property "Reference" "#FLG0101" (id 0) (at 130.81 29.845 0)
       (effects (font (size 1.27 1.27)) hide)
     )
-    (property "Value" "PWR_FLAG" (id 1) (at 130.81 28.1455 0))
+    (property "Value" "PWR_FLAG" (id 1) (at 137.16 31.75 0))
     (property "Footprint" "" (id 2) (at 130.81 31.75 0)
       (effects (font (size 1.27 1.27)) hide)
@@
   )
   (symbol (lib_id "Device:R") (at 143.51 21.59 90) (unit 1)
-    (in_bom yes) (on_board yes) (fields_autoplaced)
-    (property "Reference" "R3" (id 0) (at 143.51 16.6075 90))
+    (in_bom yes) (on_board yes)
+    (property "Reference" "R3" (id 0) (at 143.51 21.59 90))
     (property "Value" "R" (id 1) (at 143.51 19.3826 90))
     (property "Footprint" "Resistor_THT:R_Axial_DIN0207_L6.3mm_D2.5mm_P7.62mm_Horizontal" (id 2) (at 143.51 23.368 90)
@@
       (reference "J4") (unit 1) (value "UART") (footprint "Connector_PinHeader_2.54mm:PinHeader_1x04_P2.54mm_Vertical")
     )
+    (path "/00000000-0000-0000-0000-00005e9c5ed6"
+      (reference "NU1") (unit 1) (value "Numitron_IV-9") (footprint "Numitron:numitron iv-9")
+    )
+    (path "/00000000-0000-0000-0000-00005e97b8a8"
+      (reference "NU2") (unit 1) (value "Numitron_IV-9") (footprint "Numitron:numitron iv-9")
+    )
+    (path "/00000000-0000-0000-0000-00005e9c5918"
+      (reference "NU3") (unit 1) (value "Numitron_IV-9") (footprint "Numitron:numitron iv-9")
+    )
+    (path "/00000000-0000-0000-0000-00005e9c51b9"
+      (reference "NU4") (unit 1) (value "Numitron_IV-9") (footprint "Numitron:numitron iv-9")
+    )
     (path "/30f6ac74-f501-4148-81d0-578662cc8067"
       (reference "R1") (unit 1) (value "R") (footprint "Resistor_THT:R_Axial_DIN0207_L6.3mm_D2.5mm_P7.62mm_Horizontal")
@@
       (reference "SW3") (unit 1) (value "Set H") (footprint "Button_Switch_SMD:SW_SPST_CK_RS282G05A3")
     )
+    (path "/00000000-0000-0000-0000-00005e9c7f81"
+      (reference "U1") (unit 1) (value "TPIC6595") (footprint "Package_DIP:DIP-20_W7.62mm_LongPads")
+    )
     (path "/00000000-0000-0000-0000-00005e97c241"
-      (reference "U1") (unit 1) (value "TPIC6595") (footprint "Package_DIP:DIP-20_W7.62mm_LongPads")
+      (reference "U2") (unit 1) (value "TPIC6595") (footprint "Package_DIP:DIP-20_W7.62mm_LongPads")
     )
     (path "/00000000-0000-0000-0000-00005e9c63f8"
-      (reference "U2") (unit 1) (value "TPIC6595") (footprint "Package_DIP:DIP-20_W7.62mm_LongPads")
-    )
-    (path "/00000000-0000-0000-0000-00005e9c7f81"
       (reference "U3") (unit 1) (value "TPIC6595") (footprint "Package_DIP:DIP-20_W7.62mm_LongPads")
     )
@@
       (reference "U5") (unit 1) (value "ATmega8L-8A") (footprint "Package_QFP:TQFP-32_7x7mm_P0.8mm")
     )
-    (path "/00000000-0000-0000-0000-00005e9c51b9"
-      (reference "U9") (unit 1) (value "Numitron_IV-9") (footprint "Numitron:numitron iv-9")
-    )
-    (path "/00000000-0000-0000-0000-00005e9c5918"
-      (reference "U10") (unit 1) (value "Numitron_IV-9") (footprint "Numitron:numitron iv-9")
-    )
-    (path "/00000000-0000-0000-0000-00005e9c5ed6"
-      (reference "U12") (unit 1) (value "Numitron_IV-9") (footprint "Numitron:numitron iv-9")
-    )
-    (path "/00000000-0000-0000-0000-00005e97b8a8"
-      (reference "U22") (unit 1) (value "Numitron_IV-9") (footprint "Numitron:numitron iv-9")
-    )
     (path "/4bbc4b09-c5b2-44fa-801a-72cc983f0633"
